File: stim/stim.kicad_pcb (KiCad board)
At the start: 0 parts

Commit message: Upd sch & pcb
Parts:
- added C1: 100n, Capacitor_SMD:C_0603_1608Metric, F.Cu at (233.7, 161.2)
- added C2: 100n, Capacitor_SMD:C_0603_1608Metric, F.Cu at (251.5, 73.6)
- added C3: 100n, Capacitor_SMD:C_0603_1608Metric, F.Cu at (251.5, 131.9)
- added C4: 100n, Capacitor_SMD:C_0603_1608Metric, F.Cu at (251.5, 187.9)
- added C5: 100n, Capacitor_SMD:C_0603_1608Metric, F.Cu at (231.1, 73.5)
- added C6: 100n, Capacitor_SMD:C_0603_1608Metric, F.Cu at (231.1, 132.0)
- added C7: 100n, Capacitor_SMD:C_0603_1608Metric, F.Cu at (231.1, 187.8)
- added C8: 100n, Capacitor_SMD:C_0603_1608Metric, F.Cu at (240.0, 99.0)
- added C9: 100n, Capacitor_SMD:C_0603_1608Metric, F.Cu at (240.0, 109.2)
- added D1: LED, LED_SMD:LED_0805_2012Metric, F.Cu at (178.3, 203.7)
- added F1: 1.8A, Fuse:Fuse_1206_3216Metric, F.Cu at (168.4, 195.6)
- added J1: Conn_01x16, TerminalBlock_Phoenix:TerminalBlock_Phoenix_MKDS-1,5-16-5.08_1x16_P5.08mm_Horizontal, F.Cu at (293.0, 127.5)
- added J10: Conn_01x01, MountingHole:MountingHole_3.2mm_M3_Pad_Via, F.Cu at (208.5, 129.5)
- added J11: Conn_01x01, MountingHole:MountingHole_3.2mm_M3_Pad_Via, F.Cu at (305.9, 50.5)
- added J12: Conn_01x01, MountingHole:MountingHole_3.2mm_M3_Pad_Via, F.Cu at (208.0, 208.5)
- added J13: Conn_01x01, MountingHole:MountingHole_3.2mm_M3_Pad_Via, F.Cu at (130.5, 50.5)
- added J14: Conn_01x01, MountingHole:MountingHole_3.2mm_M3_Pad_Via, F.Cu at (208.5, 50.5)
- added J15: Conn_01x01, MountingHole:MountingHole_3.2mm_M3_Pad_Via, F.Cu at (130.5, 129.5)
- added J16: Conn_01x01, MountingHole:MountingHole_3.2mm_M3_Pad_Via, F.Cu at (305.9, 208.5)
- added J17: Conn_01x01, MountingHole:MountingHole_3.2mm_M3_Pad_Via, F.Cu at (130.5, 208.5)
- added J2: Conn_01x16, TerminalBlock_Phoenix:TerminalBlock_Phoenix_MKDS-1,5-16-5.08_1x16_P5.08mm_Horizontal, F.Cu at (267.9, 168.1)
- added J3: Conn_01x16, TerminalBlock_Phoenix:TerminalBlock_Phoenix_MKDS-1,5-16-5.08_1x16_P5.08mm_Horizontal, F.Cu at (293.0, 208.8)
- added J4: Conn_01x01, Connector_Wire:SolderWire-0.75sqmm_1x01_D1.25mm_OD2.3mm, F.Cu at (248.6, 208.8)
- added J5: Conn_01x02, TerminalBlock_Phoenix:TerminalBlock_Phoenix_MKDS-1,5-2-5.08_1x02_P5.08mm_Horizontal, F.Cu at (167.0, 203.8)
- added J6: Conn_01x04, TerminalBlock_Phoenix:TerminalBlock_Phoenix_MKDS-1,5-4-5.08_1x04_P5.08mm_Horizontal, F.Cu at (267.9, 188.5)
- added J7: Conn_01x04, TerminalBlock_Phoenix:TerminalBlock_Phoenix_MKDS-1,5-4-5.08_1x04_P5.08mm_Horizontal, F.Cu at (267.9, 86.9)
- added J8: Conn_01x04, TerminalBlock_Phoenix:TerminalBlock_Phoenix_MKDS-1,5-4-5.08_1x04_P5.08mm_Horizontal, F.Cu at (267.9, 66.5)
- added J9: Conn_01x04, TerminalBlock_Phoenix:TerminalBlock_Phoenix_MKDS-1,5-4-5.08_1x04_P5.08mm_Horizontal, F.Cu at (267.9, 208.8)
- added R1: 1.2k, Resistor_SMD:R_1206_3216Metric, F.Cu at (247.7, 93.9)
- added R10: 4.7k, Resistor_SMD:R_0603_1608Metric, F.Cu at (239.9, 155.4)
- added R11: 1.5k, Resistor_SMD:R_0603_1608Metric, F.Cu at (243.7, 155.4)
- added R12: 1.2k, Resistor_SMD:R_1206_3216Metric, F.Cu at (247.7, 107.9)
- added R13: 4.7k, Resistor_SMD:R_0603_1608Metric, F.Cu at (178.3, 207.3)
- added R2: 1.2k, Resistor_SMD:R_1206_3216Metric, F.Cu at (247.7, 97.8)
- added R3: 1.2k, Resistor_SMD:R_1206_3216Metric, F.Cu at (247.7, 104.1)
- added R4: 4.7k, Resistor_SMD:R_0603_1608Metric, F.Cu at (227.3, 155.4)
- added R5: 1.5k, Resistor_SMD:R_0603_1608Metric, F.Cu at (223.5, 155.4)
- added R6: 4.7k, Resistor_SMD:R_0603_1608Metric, F.Cu at (227.4, 159.5)
- added R7: 1.5k, Resistor_SMD:R_0603_1608Metric, F.Cu at (223.6, 159.5)
- added R8: 4.7k, Resistor_SMD:R_0603_1608Metric, F.Cu at (239.9, 159.5)
- added R9: 1.5k, Resistor_SMD:R_0603_1608Metric, F.Cu at (243.7, 159.5)
- added RN1: 0, Resistor_SMD:R_Array_Convex_4x0603, F.Cu at (218.4, 60.9)
- added RN10: 0, Resistor_SMD:R_Array_Convex_4x0603, F.Cu at (226.1, 175.2)
- added RN11: 0, Resistor_SMD:R_Array_Convex_4x0603, F.Cu at (226.1, 195.5)
- added RN12: 0, Resistor_SMD:R_Array_Convex_4x0603, F.Cu at (218.4, 195.5)
- added RN13: 10k, Resistor_SMD:R_Array_Convex_4x0603, F.Cu at (224.9, 96.7)
- added RN14: 10k, Resistor_SMD:R_Array_Convex_4x0603, F.Cu at (224.9, 103.0)
- added RN2: 0, Resistor_SMD:R_Array_Convex_4x0603, F.Cu at (226.1, 60.9)
- added RN3: 0, Resistor_SMD:R_Array_Convex_4x0603, F.Cu at (226.1, 81.2)
- added RN4: 0, Resistor_SMD:R_Array_Convex_4x0603, F.Cu at (218.4, 81.2)
- added RN5: 0, Resistor_SMD:R_Array_Convex_4x0603, F.Cu at (218.4, 119.3)
- added RN6: 0, Resistor_SMD:R_Array_Convex_4x0603, F.Cu at (226.1, 119.3)
- added RN7: 0, Resistor_SMD:R_Array_Convex_4x0603, F.Cu at (226.1, 139.7)
- added RN8: 0, Resistor_SMD:R_Array_Convex_4x0603, F.Cu at (218.4, 139.7)
- added RN9: 0, Resistor_SMD:R_Array_Convex_4x0603, F.Cu at (218.4, 175.2)
- added U1: OPA4192IPW, Package_SO:TSSOP-14_4.4x5mm_P0.65mm, F.Cu at (233.7, 157.4)
- added U10: ULN2003A, Package_SO:SOIC-16_3.9x9.9mm_P1.27mm, F.Cu at (217.2, 99.0)
- added U11: NUCLEO-F429ZI, lib:MODULE_NUCLEO-F429ZI, F.Cu at (169.5, 125.7)
- added U2: CD4067BM96, Package_SO:SOIC-24W_7.5x15.4mm_P1.27mm, F.Cu at (241.3, 71.1)
- added U3: CD4067BM96, Package_SO:SOIC-24W_7.5x15.4mm_P1.27mm, F.Cu at (241.3, 129.5)
- added U4: CD4067BM96, Package_SO:SOIC-24W_7.5x15.4mm_P1.27mm, F.Cu at (241.3, 185.4)
- added U5: CD4067BM96, Package_SO:SOIC-24W_7.5x15.4mm_P1.27mm, F.Cu at (221.0, 71.1)
- added U6: CD4067BM96, Package_SO:SOIC-24W_7.5x15.4mm_P1.27mm, F.Cu at (221.0, 129.5)
- added U7: CD4067BM96, Package_SO:SOIC-24W_7.5x15.4mm_P1.27mm, F.Cu at (221.0, 185.4)
- added U8: TC4427, Package_SO:SOIC-8_3.9x4.9mm_P1.27mm, F.Cu at (240.0, 95.2)
- added U9: TC4427, Package_SO:SOIC-8_3.9x4.9mm_P1.27mm, F.Cu at (240.0, 105.4)
Routing:
- net +12V: track 0.00 -> 678.1 mm, vias 0 -> 11
- net /A3: track 0.00 -> 221.4 mm, vias 0 -> 4
- net /OFF: track 0.00 -> 205.6 mm, vias 0 -> 4
- net /A1: track 0.00 -> 205.3 mm, vias 0 -> 4
- net /A0: track 0.00 -> 200.2 mm, vias 0 -> 4
- net /A2: track 0.00 -> 198.5 mm, vias 0 -> 4
- net /TST49: track 0.00 -> 133.7 mm, vias 0 -> 4
- net /TST16: track 0.00 -> 132.6 mm, vias 0 -> 2
- net /TST33: track 0.00 -> 131.0 mm, vias 0 -> 2
- net /TST15: track 0.00 -> 125.5 mm, vias 0 -> 2
- net /TST34: track 0.00 -> 124.0 mm, vias 0 -> 2
- net /TST14: track 0.00 -> 118.5 mm, vias 0 -> 2
- net /TST35: track 0.00 -> 117.1 mm, vias 0 -> 2
- net /TST13: track 0.00 -> 111.7 mm, vias 0 -> 2
- net Net-(U1-Pad3): track 0.00 -> 111.7 mm, vias 0 -> 2
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- added copper zone on B.Cu, net GND
- added copper zone on F.Cu, net GND
Other:
- board outline added: 182.5 x 165 mm
- copper layers 0 -> 2
- board text added: "+12"
- board text added: "1"
- board text added: "10"
- board text added: "11"
- board text added: "12"
- board text added: "13"
- board text added: "14"
- board text added: "15"
- board text added: "16"
- board text added: "17"
- board text added: "18"
- board text added: "19"
- board text added: "2"
- board text added: "20"
- board text added: "21"
- board text added: "22"
- board text added: "23"
- board text added: "24"
- board text added: "25"
- board text added: "26"
- board text added: "27"
- board text added: "28"
- board text added: "29"
- board text added: "3"
- board text added: "30"
- board text added: "31"
- board text added: "32"
- board text added: "33"
- board text added: "34"
- board text added: "35"
- board text added: "36"
- board text added: "37"
- board text added: "38"
- board text added: "39"
- board text added: "4"
- board text added: "40"
- board text added: "41"
- board text added: "42"
- board text added: "43"
- board text added: "44"
- board text added: "45"
- board text added: "46"
- board text added: "47"
- board text added: "48"
- board text added: "49"
- board text added: "5"
- board text added: "6"
- board text added: "7"
- board text added: "8"
- board text added: "9"
- board text added: "GND"
