File: stim/stim.kicad_sch (KiCad schematic)
At the start: 38 parts, among them U1 OPA4192IPW, U2 CD4067BM96, U3 CD4067BM96, U4 CD4067BM96, U5 CD4067BM96, U6 CD4067BM96, U7 CD4067BM96, U8 TC4427, U9 TC4427

Commit message: Upd sch & pcb
Parts:
- removed U?: ULN2003A, Package_SO:SOIC-16_3.9x9.9mm_P1.27mm, symbol Transistor_Array:ULN2003A
- added D1: LED, LED_SMD:LED_0805_2012Metric, symbol Device:LED
- added F1: 1.8A, Fuse:Fuse_1206_3216Metric, symbol Device:Fuse
- added J1, J2, J3: Conn_01x16, TerminalBlock_Phoenix:TerminalBlock_Phoenix_MKDS-1,5-16-5.08_1x16_P5.08mm_Horizontal, symbol Connector_Generic:Conn_01x16
- added J10, J11, J12, J13, J14, J15, J16, J17: Conn_01x01, MountingHole:MountingHole_3.2mm_M3_Pad_Via, symbol Connector_Generic:Conn_01x01
- added J4: Conn_01x01, Connector_Wire:SolderWire-0.75sqmm_1x01_D1.25mm_OD2.3mm, symbol Connector_Generic:Conn_01x01
- added J5: Conn_01x02, TerminalBlock_Phoenix:TerminalBlock_Phoenix_MKDS-1,5-2-5.08_1x02_P5.08mm_Horizontal, symbol Connector_Generic:Conn_01x02
- added J6, J7, J8, J9: Conn_01x04, TerminalBlock_Phoenix:TerminalBlock_Phoenix_MKDS-1,5-4-5.08_1x04_P5.08mm_Horizontal, symbol Connector_Generic:Conn_01x04
- added R10, R13, R4, R6, R8: 4.7k, Resistor_SMD:R_0603_1608Metric, symbol Device:R
- added R11, R5, R7, R9: 1.5k, Resistor_SMD:R_0603_1608Metric, symbol Device:R
- added U11: NUCLEO-F429ZI, lib:MODULE_NUCLEO-F429ZI, symbol NUCLEO-F429ZI:NUCLEO-F429ZI
- RN13, RN14: renamed from RN?; LCSC C110924 -> C29718
- gave numbers to parts that had none: 11
Connections:
- net A10 is gone; now on net A2: U4.14 (C), U7.14 (C)
- net A11 is gone; now on net A3: U4.13 (D), U7.13 (D)
- net A4 is gone; now on net A0: U3.10 (A), U6.10 (A)
- net A5 is gone; now on net A1: U3.11 (B), U6.11 (B)
- net A6 is gone; now on net A2: U3.14 (C), U6.14 (C)
- net A7 is gone; now on net A3: U3.13 (D), U6.13 (D)
- net A8 is gone; now on net A0: U4.10 (A), U7.10 (A)
- net A9 is gone; now on net A1: U4.11 (B), U7.11 (B)
- net +12V: now also RN13.1 (R1.1), RN13.2 (R2.1), RN13.3 (R3.1), RN13.4 (R4.1), RN14.4 (R4.1), D1.2 (A), F1.1, J8.1 (Pin_1), J8.2 (Pin_2), J8.3 (Pin_3), J8.4 (Pin_4), J9.1 (Pin_1), J9.2 (Pin_2), J9.3 (Pin_3), J9.4 (Pin_4), U11.CN11_24 (VIN)
- net A0: now also RN13.5 (R4.2), U10.16 (O1)
- net A1: now also RN13.6 (R3.2), U10.15 (O2)
- net A2: now also RN13.7 (R2.2), U10.14 (O3)
- net A3: now also RN13.8 (R1.2), U10.13 (O4)
- net GND: now also U10.6 (I6), U10.7 (I7), J10.1 (Pin_1), J11.1 (Pin_1), J12.1 (Pin_1), J13.1 (Pin_1), J14.1 (Pin_1), J15.1 (Pin_1), J16.1 (Pin_1), J17.1 (Pin_1), J5.2 (Pin_2), J6.1 (Pin_1), J6.2 (Pin_2), J6.3 (Pin_3), J6.4 (Pin_4), J7.1 (Pin_1), J7.2 (Pin_2), J7.3 (Pin_3), J7.4 (Pin_4), R11.1, R13.1, R5.1, R7.1, R9.1, U11.CN10_17 (GND_CN10), U11.CN10_22 (GND_CN10), U11.CN10_27 (GND_CN10), U11.CN10_3 (AGND_CN10), U11.CN10_5 (GND_CN10), U11.CN11_19 (GND_CN11), U11.CN11_20 (GND_CN11), U11.CN11_22 (GND_CN11), U11.CN11_49 (GND_CN11), U11.CN11_60 (GND_CN11), U11.CN11_71 (GND_CN11), U11.CN11_72 (GND_CN11), U11.CN11_8 (GND_CN11), U11.CN12_20 (GND_CN12), U11.CN12_32 (AGND_CN12), U11.CN12_39 (GND_CN12), U11.CN12_54 (GND_CN12), U11.CN12_63 (GND_CN12), U11.CN12_71 (GND_CN12), U11.CN12_72 (GND_CN12), U11.CN12_9 (GND_CN12), U11.CN7_8 (GND_CN7), U11.CN8_11 (GND_CN8), U11.CN8_13 (GND_CN8), U11.CN9_12 (GND_CN9), U11.CN9_23 (GND_CN9)
- net OFF: now also RN14.5 (R4.2), U10.12 (O5)
- net TST1: now also RN1.8 (R1.2), U2.9 (X0), J1.16 (Pin_16); no longer U8.4 (IN_B)
- net TST2: now also RN1.7 (R2.2), U2.8 (X1), J1.15 (Pin_15); no longer U9.2 (IN_A)
- net TST3: now also RN1.6 (R3.2), U2.7 (X2), J1.14 (Pin_14); no longer U9.4 (IN_B)
- net ADR0: now reaches U10.1 (I1)
- net ADR0: now also U11.CN12_2 (PC8)
- net at U10.10 (O7): no longer RN14.7 (R2.2)
- net at U10.11 (O6): no longer RN14.6 (R3.2)
- net ADR1: now reaches U10.2 (I2)
- net ADR1: now also U11.CN12_4 (PC6)
- net ADR2: now reaches U10.3 (I3)
- net ADR2: now also U11.CN12_6 (PC5)
- net ADR3: now reaches U10.4 (I4)
- net ADR3: now also U11.CN12_13 (PA6)
- net MUX_OFF: now reaches U10.5 (I5)
- net MUX_OFF: now also U11.CN12_15 (PA7)
- net at U6.6 (X3): now also RN5.8 (R1.2); no longer RN5.1 (R1.1)
- net at U6.7 (X2): now also RN5.7 (R2.2); no longer RN5.2 (R2.1)
- net at U6.8 (X1): now also RN5.6 (R3.2); no longer RN5.3 (R3.1)
- net at U6.9 (X0): now also RN5.5 (R4.2); no longer RN5.4 (R4.1)
- net TST17: now reaches U3.9 (X0)
- net TST17: now also RN5.4 (R4.1), J2.16 (Pin_16); no longer RN5.5 (R4.2)
- net TST18: now reaches U3.8 (X1)
- net TST18: now also RN5.3 (R3.1), J2.15 (Pin_15); no longer RN5.6 (R3.2)
- net TST19: now reaches U3.7 (X2)
- net TST19: now also RN5.2 (R2.1), J2.14 (Pin_14); no longer RN5.7 (R2.2)
- net TST20: now reaches U3.6 (X3)
- net TST20: now also RN5.1 (R1.1), J2.13 (Pin_13); no longer RN5.8 (R1.2)
- net at U1.12 (+): now also U3.1 (X); no longer R12.1
- net at RN12.8 (R1.2): now also U7.16 (X15); no longer U4.16 (X15)
- net at RN12.7 (R2.2): now also U7.17 (X14); no longer U4.17 (X14)
- net at RN12.6 (R3.2): now also U7.18 (X13); no longer U4.18 (X13)
- net at RN12.5 (R4.2): now also U7.19 (X12); no longer U4.19 (X12)
- net at RN10.8 (R1.2): now also U7.2 (X7); no longer U4.2 (X7)
- net at RN11.8 (R1.2): now also U7.20 (X11); no longer U4.20 (X11)
- net at RN11.7 (R2.2): now also U7.21 (X10); no longer U4.21 (X10)
- net at RN11.6 (R3.2): now also U7.22 (X9); no longer U4.22 (X9)
- net at RN11.5 (R4.2): now also U7.23 (X8); no longer U4.23 (X8)
- net at RN10.7 (R2.2): now also U7.3 (X6); no longer U4.3 (X6)
- net at RN10.6 (R3.2): now also U7.4 (X5); no longer U4.4 (X5)
- net at RN10.5 (R4.2): now also U7.5 (X4); no longer U4.5 (X4)
- net at RN9.8 (R1.2): now also U7.6 (X3); no longer U4.6 (X3)
- net at RN9.7 (R2.2): now also U7.7 (X2); no longer U4.7 (X2)
- net at RN9.6 (R3.2): now also U7.8 (X1); no longer U4.8 (X1)
- net at RN9.5 (R4.2): now also U7.9 (X0); no longer U4.9 (X0)
- net at U6.20 (X11): now also RN7.8 (R1.2); no longer RN7.1 (R1.1)
- net at U6.21 (X10): now also RN7.7 (R2.2); no longer RN7.2 (R2.1)
- net at U6.22 (X9): now also RN7.6 (R3.2); no longer RN7.3 (R3.1)
- net at U6.23 (X8): now also RN7.5 (R4.2); no longer RN7.4 (R4.1)
- net TST25: now reaches U3.23 (X8)
- net TST25: now also RN7.4 (R4.1), J2.8 (Pin_8); no longer RN7.5 (R4.2)
- net TST26: now reaches U3.22 (X9)
- net TST26: now also RN7.3 (R3.1), J2.7 (Pin_7); no longer RN7.6 (R3.2)
- net TST27: now reaches U3.21 (X10)
- net TST27: now also RN7.2 (R2.1), J2.6 (Pin_6); no longer RN7.7 (R2.2)
- net TST28: now reaches U3.20 (X11)
- net TST28: now also RN7.1 (R1.1), J2.5 (Pin_5); no longer RN7.8 (R1.2)
- net TST40: now reaches RN10.1 (R1.1)
- net TST40: now also U4.2 (X7), J3.9 (Pin_9); no longer U7.2 (X7)
- net TST39: now reaches RN10.2 (R2.1)
- net TST39: now also U4.3 (X6), J3.10 (Pin_10); no longer U7.3 (X6)
- net TST38: now reaches RN10.3 (R3.1)
- net TST38: now also U4.4 (X5), J3.11 (Pin_11); no longer U7.4 (X5)
- net TST37: now reaches RN10.4 (R4.1)
- net TST37: now also U4.5 (X4), J3.12 (Pin_12); no longer U7.5 (X4)
- net at RN1.1 (R1.1): now also U5.9 (X0); no longer U5.6 (X3)
- net at RN1.2 (R2.1): now also U5.8 (X1); no longer U5.7 (X2)
- net at RN1.3 (R3.1): now also U5.7 (X2); no longer U5.8 (X1)
- net at RN1.4 (R4.1): now also U5.6 (X3); no longer U5.9 (X0)
- net TST4: now reaches RN1.5 (R4.2)
- net TST4: now also U2.6 (X3), J1.13 (Pin_13); no longer U2.9 (X0)
- net at U6.16 (X15): now also RN8.8 (R1.2); no longer RN8.1 (R1.1)
- net at U6.17 (X14): now also RN8.7 (R2.2); no longer RN8.2 (R2.1)
- net at U6.18 (X13): now also RN8.6 (R3.2); no longer RN8.3 (R3.1)
- net at U6.19 (X12): now also RN8.5 (R4.2); no longer RN8.4 (R4.1)
- net at U6.2 (X7): now also RN6.8 (R1.2); no longer RN6.1 (R1.1)
- net at U6.3 (X6): now also RN6.7 (R2.2); no longer RN6.2 (R2.1)
- net at U6.4 (X5): now also RN6.6 (R3.2); no longer RN6.3 (R3.1)
- net at U6.5 (X4): now also RN6.5 (R4.2); no longer RN6.4 (R4.1)
- net TST48: now reaches RN12.1 (R1.1)
- net TST48: now also U4.16 (X15), J3.1 (Pin_1); no longer U7.16 (X15)
- net TST47: now reaches RN12.2 (R2.1)
- net TST47: now also U4.17 (X14), J3.2 (Pin_2); no longer U7.17 (X14)
- net TST46: now reaches RN12.3 (R3.1)
- net TST46: now also U4.18 (X13), J3.3 (Pin_3); no longer U7.18 (X13)
- net TST45: now reaches RN12.4 (R4.1)
- net TST45: now also U4.19 (X12), J3.4 (Pin_4); no longer U7.19 (X12)
- net TST49: now reaches U1.5 (+)
- net TST49: now also R12.1, J4.1 (Pin_1); no longer U3.1 (X)
- net TST32: now reaches U3.16 (X15)
- net TST32: now also RN8.1 (R1.1), J2.1 (Pin_1); no longer RN8.8 (R1.2)
- net TST31: now reaches U3.17 (X14)
- net TST31: now also RN8.2 (R2.1), J2.2 (Pin_2); no longer RN8.7 (R2.2)
- net TST30: now reaches U3.18 (X13)
- net TST30: now also RN8.3 (R3.1), J2.3 (Pin_3); no longer RN8.6 (R3.2)
- net TST29: now reaches U3.19 (X12)
- net TST29: now also RN8.4 (R4.1), J2.4 (Pin_4); no longer RN8.5 (R4.2)
- net TST24: now reaches U3.2 (X7)
- net TST24: now also RN6.1 (R1.1), J2.9 (Pin_9); no longer RN6.8 (R1.2)
- net TST23: now reaches U3.3 (X6)
- net TST23: now also RN6.2 (R2.1), J2.10 (Pin_10); no longer RN6.7 (R2.2)
- net TST22: now reaches U3.4 (X5)
- net TST22: now also RN6.3 (R3.1), J2.11 (Pin_11); no longer RN6.6 (R3.2)
- net TST21: now reaches U3.5 (X4)
- net TST21: now also RN6.4 (R4.1), J2.12 (Pin_12); no longer RN6.5 (R4.2)
- net at U1.1, U1.2 (-): now also R4.2
- net at RN3.1 (R1.1): now also U5.23 (X8); no longer U5.20 (X11)
- net at RN3.2 (R2.1): now also U5.22 (X9); no longer U5.21 (X10)
- net at RN3.3 (R3.1): now also U5.21 (X10); no longer U5.22 (X9)
- net at RN3.4 (R4.1): now also U5.20 (X11); no longer U5.23 (X8)
- net TST12: now reaches RN3.5 (R4.2)
- net TST12: now also U2.20 (X11), J1.5 (Pin_5); no longer U2.23 (X8)
- net TST10: now reaches U2.22 (X9)
- net TST10: now also RN3.7 (R2.2), J1.7 (Pin_7); no longer RN3.6 (R3.2)
- net TST11: now reaches U2.21 (X10)
- net TST11: now also RN3.6 (R3.2), J1.6 (Pin_6); no longer RN3.7 (R2.2)
- net TST9: now reaches RN3.8 (R1.2)
- net TST9: now also U2.23 (X8), J1.8 (Pin_8); no longer U2.20 (X11)
- net at RN4.1 (R1.1): now also U5.19 (X12); no longer U5.16 (X15)
- net at RN4.2 (R2.1): now also U5.18 (X13); no longer U5.17 (X14)
- net at RN4.3 (R3.1): now also U5.17 (X14); no longer U5.18 (X13)
- net at RN4.4 (R4.1): now also U5.16 (X15); no longer U5.19 (X12)
- net TST13: now reaches U2.19 (X12)
- net TST13: now also RN4.8 (R1.2), J1.4 (Pin_4); no longer RN4.5 (R4.2)
- net TST14: now reaches U2.18 (X13)
- net TST14: now also RN4.7 (R2.2), J1.3 (Pin_3); no longer RN4.6 (R3.2)
- net TST15: now reaches U2.17 (X14)
- net TST15: now also RN4.6 (R3.2), J1.2 (Pin_2); no longer RN4.7 (R2.2)
- net TST16: now reaches U2.16 (X15)
- net TST16: now also RN4.5 (R4.2), J1.1 (Pin_1); no longer RN4.8 (R1.2)
- net TST36: now reaches RN9.1 (R1.1)
- net TST36: now also U4.6 (X3), J3.13 (Pin_13); no longer U7.6 (X3)
- net TST35: now reaches RN9.2 (R2.1)
- net TST35: now also U4.7 (X2), J3.14 (Pin_14); no longer U7.7 (X2)
- net TST34: now reaches RN9.3 (R3.1)
- net TST34: now also U4.8 (X1), J3.15 (Pin_15); no longer U7.8 (X1)
- net TST33: now reaches RN9.4 (R4.1)
- net TST33: now also U4.9 (X0), J3.16 (Pin_16); no longer U7.9 (X0)
- net TST5: now reaches RN2.8 (R1.2)
- net TST5: now also U2.5 (X4), J1.12 (Pin_12); no longer U2.2 (X7)
- net TST6: now reaches RN2.7 (R2.2)
- net TST6: now also U2.4 (X5), J1.11 (Pin_11); no longer U2.3 (X6)
- net TST7: now reaches RN2.6 (R3.2)
- net TST7: now also U2.3 (X6), J1.10 (Pin_10); no longer U2.4 (X5)
- net TST8: now reaches RN2.5 (R4.2)
- net TST8: now also U2.2 (X7), J1.9 (Pin_9); no longer U2.5 (X4)
- net at U1.6 (-), U1.7: now also R6.2
- net at U1.8, U1.9 (-): now also R8.2
- net at U5.2 (X7): now also RN2.4 (R4.1); no longer RN2.1 (R1.1)
- net at U5.3 (X6): now also RN2.3 (R3.1); no longer RN2.2 (R2.1)
- net at U5.4 (X5): now also RN2.2 (R2.1); no longer RN2.3 (R3.1)
- net at U5.5 (X4): now also RN2.1 (R1.1); no longer RN2.4 (R4.1)
- net at U1.13 (-), U1.14: now also R10.2
- net TST44: now reaches RN11.1 (R1.1)
- net TST44: now also U4.20 (X11), J3.5 (Pin_5); no longer U7.20 (X11)
- net TST43: now reaches RN11.2 (R2.1)
- net TST43: now also U4.21 (X10), J3.6 (Pin_6); no longer U7.21 (X10)
- net TST42: now reaches RN11.3 (R3.1)
- net TST42: now also U4.22 (X9), J3.7 (Pin_7); no longer U7.22 (X9)
- net TST41: now reaches RN11.4 (R4.1)
- net TST41: now also U4.23 (X8), J3.8 (Pin_8); no longer U7.23 (X8)
- net TST0 renamed OUT0
- net OUT0: now also U11.CN12_16 (PB12)
- new net: D1.1 (K), R13.2
- new net: F1.2, J5.1 (Pin_1)
- new net: U11.CN11_10 (NC), U11.CN11_26 (NC), U11.CN11_67 (NC)
- new net IN0: R4.1, R5.2, U11.CN12_38 (PF4)
- new net IN1: R10.1, R11.2, U11.CN12_36 (PF5)
- new net IN2: R8.1, R9.2, U11.CN12_58 (PF3)
- new net IN3: R6.1, R7.2, U11.CN12_42 (PF10)
- new net OUT1: U11.CN12_18 (PB11), U8.4 (IN_B)
- new net OUT2: U11.CN12_19 (PC7), U9.2 (IN_A)
- new net OUT3: U11.CN12_34 (PC4), U9.4 (IN_B)
Other:
- moved on the sheet: RN10, RN11, RN12, RN13, RN14, RN5, RN6, RN7, RN8, RN9, U10, U1B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
