File: digital_inputs/digital_inputs.kicad_pcb (KiCad board)
At the start: 2 copper layers, 182.5 x 165 mm, 66 parts, among them J1 Conn_01x16, J10 Conn_01x01, J11 Conn_01x01, J12 Conn_01x01, J13 Conn_01x01, J14 Conn_01x01, J15 Conn_01x01, J16 Conn_01x01, J17 Conn_01x01, J2 Conn_01x16, J3 Conn_01x16, J4 Conn_01x01, J5 Conn_01x02, J6 Conn_01x04, J7 Conn_01x04, J8 Conn_01x04, J9 Conn_01x04, U1 OPA4192IPW, U10 ULN2003A, U11 NUCLEO-F429ZI, U2 CD4067BM96, U3 CD4067BM96, U4 CD4067BM96, U5 CD4067BM96, U6 CD4067BM96, U7 CD4067BM96, U8 TC4427, U9 TC4427

Commit message: Rename #8
Other:
- board text added: "Digital inputs rusefi.com"
Changed lines of the file:
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@@
     (effects (font (size 2 2) (thickness 0.3)))
+  )
+  (gr_text "Digital inputs\nrusefi.com" (at 228.8 206.3) (layer "F.SilkS")
+    (effects (font (size 3 3) (thickness 0.3)))
   )
   (gr_text "33" (at 300.64 132.58) (layer "F.SilkS")

Commit message: Fab preview
Other:
- board text added: "Digital inputs rev. a rusefi.com"
- board text removed: "Digital inputs rusefi.com"

Commit message: #14 #15
Parts:
- added C10: 47p, Capacitor_SMD:C_0603_1608Metric, F.Cu at (247.6, 36.1)
- added C11: 47p, Capacitor_SMD:C_0603_1608Metric, F.Cu at (252.3, 34.7)
- added C12: 100n, Capacitor_SMD:C_0603_1608Metric, F.Cu at (252.0, 39.5)
- added J18: Conn_01x02, TerminalBlock_Phoenix:TerminalBlock_Phoenix_MKDS-1,5-2-5.08_1x02_P5.08mm_Horizontal, F.Cu at (224.3, 36.5)
- added J19: 6437288-3, rusefi_lib1:TE_6437288-3, F.Cu at (198.2, 55.2)
- added U12: TJA1051T-3, Package_SO:SOIC-8_3.9x4.9mm_P1.27mm, F.Cu at (237.1, 33.4)
Connections:
- U11 pad CN11_16: unconnected-(U11-PadCN11_16) -> +3V3
- U11 pad CN11_18: unconnected-(U11-PadCN11_18) -> +5V
- U11 pad CN12_12: unconnected-(U11-PadCN12_12) -> /CAN_TX
- U11 pad CN12_14: unconnected-(U11-PadCN12_14) -> /CAN_RX
Other:
- board text added: "Digital inputs rev. b rusefi.com"
- board text removed: "Digital inputs rev. a rusefi.com"
