File: digital_inputs/digital_inputs.kicad_pcb (KiCad board)
At the start: 2 copper layers, 182.5 x 165 mm, 130 parts, among them J1 6437288-2, J10 Conn_01x01, J11 Conn_01x01, J12 Conn_01x01, J13 Conn_01x01, J14 Conn_01x01, J15 Conn_01x01, J16 Conn_01x01, J17 Conn_01x01, J19 6437288-3, J3 Conn_01x08, J4 Conn_01x01, J5 Conn_01x02, J6 Conn_01x04, J7 Conn_01x04, J8 Conn_01x04, J9 Conn_01x04, Q1 AO3400A, Q2 AO3400A, Q3 AO3400A, Q4 AO3400A, Q5 AO3400A, Q6 AO3400A, Q7 AO3400A, Q8 AO3400A, U1 OPA4192IPW, U10 ULN2003A, U11 NUCLEO-F429ZI, U12 TJA1051T-3, U2 CD4067BM96, U3 CD4067BM96, U4 CD4067BM96, U5 CD4067BM96, U6 CD4067BM96, U7 CD4067BM96, U8 TC4427, U9 TC4427

Commit message: Upd pcb
Parts:
- removed U11: NUCLEO-F429ZI, lib:MODULE_NUCLEO-F429ZI
- added D2: PESD1CAN, Package_TO_SOT_SMD:SOT-23, F.Cu at (281.3, 52.9)
- added H1: MountingHole, MountingHole:MountingHole_3.2mm_M3, F.Cu at (145.4, 87.0)
- added H2: MountingHole, MountingHole:MountingHole_3.2mm_M3, F.Cu at (193.6, 88.3)
- added H3: MountingHole, MountingHole:MountingHole_3.2mm_M3, F.Cu at (178.4, 139.1)
- added H4: MountingHole, MountingHole:MountingHole_3.2mm_M3, F.Cu at (146.6, 163.2)
- added H5: MountingHole, MountingHole:MountingHole_3.2mm_M3, F.Cu at (192.4, 163.2)
- added J18: Conn_02x05_Odd_Even, Connector_PinHeader_2.54mm:PinHeader_2x05_P2.54mm_Vertical, F.Cu at (137.8, 108.6)
- added J2: Conn_02x07_Odd_Even, Connector_PinHeader_2.54mm:PinHeader_2x07_P2.54mm_Vertical, F.Cu at (137.8, 90.8)
- added J20: Conn_02x24_Odd_Even, Connector_PinHeader_2.54mm:PinHeader_2x24_P2.54mm_Vertical, F.Cu at (137.8, 121.3)
- added J21: Conn_02x08_Odd_Even, Connector_PinHeader_2.54mm:PinHeader_2x08_P2.54mm_Vertical, F.Cu at (145.4, 101.0)
- added J22: Conn_02x15_Odd_Even, Connector_PinHeader_2.54mm:PinHeader_2x15_P2.54mm_Vertical, F.Cu at (145.4, 123.8)
- added J23: Conn_02x10_Odd_Even, Connector_PinHeader_2.54mm:PinHeader_2x10_P2.54mm_Vertical, F.Cu at (191.1, 91.8)
- added J24: Conn_02x17_Odd_Even, Connector_PinHeader_2.54mm:PinHeader_2x17_P2.54mm_Vertical, F.Cu at (191.1, 118.7)
- added J25: Conn_02x10_Odd_Even, Connector_PinHeader_2.54mm:PinHeader_2x10_P2.54mm_Vertical, F.Cu at (198.7, 90.8)
- added J26: Conn_02x06_Odd_Even, Connector_PinHeader_2.54mm:PinHeader_2x06_P2.54mm_Vertical, F.Cu at (198.7, 116.2)
- added J27: Conn_02x16_Odd_Even, Connector_PinHeader_2.54mm:PinHeader_2x16_P2.54mm_Vertical, F.Cu at (198.7, 131.5)
- added J28: Conn_02x04_Odd_Even, Connector_PinHeader_2.54mm:PinHeader_2x04_P2.54mm_Vertical, F.Cu at (198.7, 172.1)
- added R56: DNP, Resistor_SMD:R_0402_1005Metric, F.Cu at (278.4, 52.9)
Connections:
- net /HALL0_0 renamed /DIG_0
- net /HALL0_1 renamed /DIG_1
- net /HALL0_2 renamed /DIG_2
- net /HALL0_3 renamed /DIG_3
- net /HALL0_4 renamed /DIG_4
- net /HALL0_5 renamed /DIG_5
- net /HALL0_6 renamed /DIG_6
- net /HALL0_7 renamed /DIG_7
- net /OUT_HALL0_0 renamed /OUT_DIG_0
- net /OUT_HALL0_1 renamed /OUT_DIG_1
- net /OUT_HALL0_2 renamed /OUT_DIG_2
- net /OUT_HALL0_3 renamed /OUT_DIG_3
- net /OUT_HALL0_4 renamed /OUT_DIG_4
- net /OUT_HALL0_5 renamed /OUT_DIG_5
- net /OUT_HALL0_6 renamed /OUT_DIG_6
- net /OUT_HALL0_7 renamed /OUT_DIG_7
- U12 pad 5: +3V3 -> +3.3V
Routing:
- net +3V3: track 168.8 -> 0.00 mm, vias 1 -> 0
- net +3.3V: track 0.00 -> 168.8 mm, vias 0 -> 1
- net /MUX_OFF: track 22.7 -> 20.6 mm
- net /CAN_L: track 51.2 -> 52.8 mm
- net /CAN_H: track 47.3 -> 48.6 mm
- net GND: vias 414 -> 415

Commit message: #14 #16 #23
Parts:
- R24, R30: value 910 -> 820
- R26, R32, R39, R49: value 470 -> 820
- R27: value 100 -> 120
- R28, R43, R54, R55: value 910 -> 470
- R29: value 330 -> 100
- R31: value 470 -> 220
- R34: value 100 -> 470
- R35: value 100 -> 220
- R36: value 330 -> 820
- R37, R58: value 330 -> 510
- R38: value 910 -> 510
- R42: value 330 -> 220
- R53: value 470 -> 330
- turned R38 to 180 degrees
Connections:
- R38 pad 1: /REF12 -> /5V_2
- R38 pad 2: GND -> /REF12
- R39 pad 1: /5V_2 -> /REF12
- R39 pad 2: /REF12 -> GND
Other:
- board text added: "+12V"
- board text added: "0.5V"
- board text added: "0.6V"
- board text added: "0.8V"
- board text added: "0.9V"
- board text added: "1.1V"
- board text added: "1.4V"
- board text added: "1.6V"
- board text added: "1.9V"
- board text added: "2.1V"
- board text added: "2.5V"
- board text added: "2.9V"
- board text added: "3.1V"
- board text added: "3.4V"
- board text added: "3.8V"
- board text added: "4.1V"
- board text added: "4.5V"
- board text added: "5V_1"
- board text added: "5V_2"
- board text added: "CAN_H"
- board text added: "CAN_L"
- board text added: "OUT_D0"
- board text added: "OUT_D1"
- board text added: "OUT_D2"
- board text added: "OUT_D3"
- board text added: "OUT_D4"
- board text added: "OUT_D5"
- board text added: "OUT_D6"
- board text added: "OUT_D7"
- board text added: "PD_1k"
- board text added: "PD_2k"
- board text added: "T1"
- board text added: "T10"
- board text added: "T11"
- board text added: "T12"
- board text added: "T14"
- board text added: "T15"
- board text added: "T16"
- board text added: "T17"
- board text added: "T18"
- board text added: "T19"
- board text added: "T2"
- board text added: "T20"
- board text added: "T21"
- board text added: "T22"
- board text added: "T23"
- board text added: "T24"
- board text added: "T25"
- board text added: "T26"
- board text added: "T27"
- board text added: "T28"
- board text added: "T29"
- board text added: "T3"
- board text added: "T30"
- board text added: "T31"
- board text added: "T32"
- board text added: "T33"
- board text added: "T34"
- board text added: "T35"
- board text added: "T36"
- board text added: "T37"
- board text added: "T38"
- board text added: "T39"
- board text added: "T4"
- board text added: "T40"
- board text added: "T5"
- board text added: "T6"
- board text added: "T7"
- board text added: "T8"
- board text added: "T9"

Commit message: check
Connections:
- R38 pad 1: /5V_2 -> GND
- R39 pad 1: /REF12 -> /5V_2
- R39 pad 2: GND -> /REF12
Changed lines of the file:
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@@
       (stroke (width 0.1) (type solid)) (layer "F.Fab"))
     (pad "1" smd roundrect (at -0.825 0 180) (size 0.8 0.95) (layers "F.Cu" "F.Paste" "F.Mask") (roundrect_rratio 0.25)
-      (net 182 "/5V_2") (pintype "passive"))
+      (net 1 "GND") (pintype "passive"))
     (pad "2" smd roundrect (at 0.825 0 180) (size 0.8 0.95) (layers "F.Cu" "F.Paste" "F.Mask") (roundrect_rratio 0.25)
       (net 165 "/REF12") (pintype "passive"))
@@
       (stroke (width 0.1) (type solid)) (layer "F.Fab"))
     (pad "1" smd roundrect (at -0.825 0 180) (size 0.8 0.95) (layers "F.Cu" "F.Paste" "F.Mask") (roundrect_rratio 0.25)
-      (net 165 "/REF12") (pintype "passive"))
+      (net 182 "/5V_2") (pintype "passive"))
     (pad "2" smd roundrect (at 0.825 0 180) (size 0.8 0.95) (layers "F.Cu" "F.Paste" "F.Mask") (roundrect_rratio 0.25)
-      (net 1 "GND") (pintype "passive"))
+      (net 165 "/REF12") (pintype "passive"))
     (model "${KICAD6_3DMODEL_DIR}/Resistor_SMD.3dshapes/R_0603_1608Metric.wrl"
       (offset (xyz 0 0 0))
