File: digital_inputs/digital_inputs.kicad_pcb (KiCad board)
At the start: 2 copper layers, 182.5 x 165 mm, 170 parts, among them J1 6437288-2, J10 Conn_01x01, J11 Conn_01x01, J12 Conn_01x01, J13 Conn_01x01, J14 Conn_01x01, J15 Conn_01x01, J16 Conn_01x01, J17 Conn_01x01, J18 Conn_02x05_Odd_Even, J19 6437288-3, J2 Conn_02x07_Odd_Even, J20 Conn_02x24_Odd_Even, J21 Conn_02x08_Odd_Even, J22 Conn_02x15_Odd_Even, J23 Conn_02x10_Odd_Even, J24 Conn_02x17_Odd_Even, J25 Conn_02x10_Odd_Even, J26 Conn_02x06_Odd_Even, J27 Conn_02x16_Odd_Even, J28 Conn_02x04_Odd_Even, J3 Conn_01x08, J4 Conn_01x01, J5 Conn_01x02, J6 Conn_01x04, J7 Conn_01x04, J8 Conn_01x04, J9 Conn_01x04, P1 Pad, P10 Pad, P11 Pad, P12 Pad, P13 Pad, P14 Pad, P15 Pad, P16 Pad, P17 Pad, P2 Pad, P3 Pad, P4 Pad, P5 Pad, P6 Pad, P7 Pad, P8 Pad, P9 Pad, Q1 AO3400A, Q2 AO3400A, Q3 AO3400A, Q4 AO3400A, Q5 AO3400A, Q6 AO3400A, Q7 AO3400A, Q8 AO3400A, U1 OPA2192IDR, U10 ULN2003A, U11 OPA2192IDR, U12 TJA1051T-3, U2 CD4067BM96, U3 CD4067BM96, U4 CD4067BM96, U5 CD4067BM96, U6 CD4067BM96, U7 CD4067BM96, U8 TC4427, U9 TC4427

Commit message: Upd PCB
Parts:
- added C14: 47p, Capacitor_SMD:C_0603_1608Metric, F.Cu at (218.2, 107.0)
- added C15: 47p, Capacitor_SMD:C_0603_1608Metric, F.Cu at (218.3, 112.5)
- added C16: 100n, Capacitor_SMD:C_0603_1608Metric, F.Cu at (209.4, 104.5)
- added CB1: CircuitBreaker_1P, lib:RS601HL-1010011BB, F.Cu at (152.0, 207.7)
- added D6: PESD1CAN, Package_TO_SOT_SMD:SOT-23, F.Cu at (218.5, 109.7)
- added P18: Pad, hellen-one-common:PAD-TH, F.Cu at (224.2, 108.5)
- added P19: Pad, hellen-one-common:PAD-TH, F.Cu at (224.2, 111.6)
- added R62: DNP, Resistor_SMD:R_0603_1608Metric, F.Cu at (214.5, 109.7)
- added U13: TJA1051T-3, Package_SO:SOIC-8_3.9x4.9mm_P1.27mm, F.Cu at (209.6, 109.7)
- R56: footprint Resistor_SMD:R_0402_1005Metric -> Resistor_SMD:R_0603_1608Metric
- moved D1 34.2 mm to (144.1, 203.6)
- moved R13 34.2 mm to (144.1, 207.2)
- moved F1 11.0 mm to (161.2, 203.9), turned to 0 degrees
- moved R56 0.20 mm to (278.6, 52.9)
- moved D2 0.20 mm to (281.5, 52.9)
Connections:
- F1 pad 1: +12V -> Net-(CB1-Pad1)
- J20 pad 31: unconnected-(J20-PD1-Pad31) -> /CAN_TX
- J20 pad 33: /CAN_TX -> /CAN_RX
- J20 pad 35: /CAN_RX -> unconnected-(J20-PG0-Pad35)
- J25 pad 10: unconnected-(J25-PD8-Pad10) -> /OUT0
- J25 pad 16: /OUT0 -> /CAN2_RX
- J25 pad 17: unconnected-(J25-PB6-Pad17) -> /CAN2_TX
Routing:
- net +3.3V: track 168.8 -> 220.3 mm, vias 1 -> 4
- net +5V: track 158.6 -> 205.3 mm, vias 1 -> 4
- net +12V: track 722.1 -> 740.5 mm
- net /CAN2_L: track 0.00 -> 14.7 mm
- net /CAN2_H: track 0.00 -> 14.3 mm
- net /CAN2_TX: track 0.00 -> 11.1 mm
- net Net-(CB1-Pad1): track 0.00 -> 9.37 mm
- net /CAN2_RX: track 0.00 -> 7.14 mm
- net /OUT0: track 46.2 -> 51.4 mm
- net Net-(J5-Pin_1): track 8.26 -> 4.43 mm
- net /OUT1: track 44.4 -> 46.9 mm
- net /CAN_TX: track 199.7 -> 197.4 mm
- net /CAN_RX: track 199.2 -> 197.0 mm
- net /DIG_5: track 205.0 -> 202.9 mm
- net /OUT3: track 56.8 -> 55.1 mm
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Other:
- board text added: "H CAN2 L"

Commit message: Rev D export
Parts:
- removed J18: Conn_02x05_Odd_Even, Connector_PinHeader_2.54mm:PinHeader_2x05_P2.54mm_Vertical
- removed J2: Conn_02x07_Odd_Even, Connector_PinHeader_2.54mm:PinHeader_2x07_P2.54mm_Vertical
- added C17: 10u, Capacitor_SMD:C_0805_2012Metric, F.Cu at (147.5, 204.2)
- added C18: 10u, Capacitor_SMD:C_0805_2012Metric, F.Cu at (159.1, 199.1)
- added J29: Conn_02x10_Odd_Even, Connector_PinHeader_2.54mm:PinHeader_2x10_P2.54mm_Vertical, F.Cu at (137.8, 156.8)
- added J30: Conn_02x14_Odd_Even, Connector_PinHeader_2.54mm:PinHeader_2x16_P2.54mm_Vertical, F.Cu at (137.8, 116.2)
- added U14: LM78M05_TO252, Package_TO_SOT_SMD:TO-252-2, F.Cu at (153.0, 200.1)
- J20: value Conn_02x24_Odd_Even -> Conn_02x10_Odd_Even; footprint Connector_PinHeader_2.54mm:PinHeader_2x24_P2.54mm_Vertical -> Connector_PinHeader_2.54mm:PinHeader_2x10_P2.54mm_Vertical
- moved J20 30.5 mm to (137.8, 90.8)
- moved R13 15.0 mm to (132.1, 198.2), turned to -90 degrees
- moved D1 12.1 mm to (132.1, 201.8), turned to -90 degrees
- moved CB1 12.0 mm to (140.0, 207.7)
Connections:
- J20 pad 16: unconnected-(J20-PD3-Pad16) -> +3.3V
- J20 pad 18: unconnected-(J20-PG2-Pad18) -> +5V
- J20 pad 19: unconnected-(J20-PD6-Pad19) -> GND
- J20 pad 20: unconnected-(J20-PG3-Pad20) -> GND
- J20 pad 6: unconnected-(J20-PA1-Pad6) -> /E5V
- J20 pad 8: unconnected-(J20-PA4-Pad8) -> GND
Routing:
- net /E5V: track 0.00 -> 124.6 mm
- net +12V: track 740.5 -> 755.0 mm
- net Net-(CB1-Pad1): track 9.37 -> 21.9 mm
- net GND: vias 415 -> 429
Other:
- board text added: "Digital inputs rev D rusefi.com"
- board text removed: "Digital inputs rev С rusefi.com"
