File: digital_inputs/digital_inputs.kicad_sch (KiCad schematic)
At the start: 66 parts, among them J1 Conn_01x16, J10 Conn_01x01, J11 Conn_01x01, J12 Conn_01x01, J13 Conn_01x01, J14 Conn_01x01, J15 Conn_01x01, J16 Conn_01x01, J17 Conn_01x01, J2 Conn_01x16, J3 Conn_01x16, J4 Conn_01x01, J5 Conn_01x02, J6 Conn_01x04, J7 Conn_01x04, J8 Conn_01x04, J9 Conn_01x04, U1 OPA4192IPW, U10 ULN2003A, U11 NUCLEO-F429ZI, U2 CD4067BM96, U3 CD4067BM96, U4 CD4067BM96, U5 CD4067BM96, U6 CD4067BM96, U7 CD4067BM96, U8 TC4427, U9 TC4427

Commit message: Fab preview
Parts:
- F1: LCSC JK-nSMD100-16 -> C369161
Changed lines of the file:
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@@
       (effects (font (size 1.27 1.27)) hide)
     )
-    (property "LCSC" "JK-nSMD100-16" (id 4) (at 313.69 44.45 0)
+    (property "LCSC" "C369161" (id 4) (at 313.69 44.45 0)
       (effects (font (size 1.27 1.27)) hide)
     )

Commit message: #13
Parts:
- added C10, C11: 47p, hellen-one-common:C0603, symbol hellen-one-common:Cap
- added C12: 100n, hellen-one-common:C0603, symbol hellen-one-common:Cap
- added J18: Conn_01x02, TerminalBlock_Phoenix:TerminalBlock_Phoenix_MKDS-1,5-2-5.08_1x02_P5.08mm_Horizontal, symbol Connector_Generic:Conn_01x02
- added U12: TJA1051T-3, Package_SO:SOIC-8_3.9x4.9mm_P1.27mm, symbol Interface_CAN_LIN:TJA1051T-3
Connections:
- net GND: now also C10.2, C11.1, C12.1, U12.2 (GND), U12.8 (S)
- net CAN_TX: now reaches U11.CN12_12 (PA12)
- net CAN_TX: now also U12.1 (TXD)
- net CAN_RX: now reaches U11.CN12_14 (PA11)
- net CAN_RX: now also U12.4 (RXD)
- new net +3V3: U12.5 (VIO)
- new net +5V: C12.2, U12.3 (VCC)
- new net CAN_H: C10.1, J18.1 (Pin_1), U12.7 (CANH)
- new net CAN_L: C11.2, J18.2 (Pin_2), U12.6 (CANL)

Commit message: CAN power
Connections:
- net +3V3: now also U11.CN11_16 (+3V3)
- net +5V: now also U11.CN11_18 (+5V)
Changed lines of the file:
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@@
     (pin "1")
   )
+  (symbol (lib_id "power:+3.3V") (at 430.53 34.29 270) (mirror x) (unit 1)
+    (in_bom yes) (on_board yes)
+    (property "Reference" "#PWR?" (id 0) (at 426.72 34.29 0)
+      (effects (font (size 1.27 1.27)) hide)
+    )
+    (property "Value" "+3.3V" (id 1) (at 436.245 34.29 90))
+    (property "Footprint" "" (id 2) (at 430.53 34.29 0)
+      (effects (font (size 1.27 1.27)) hide)
+    )
+    (property "Datasheet" "" (id 3) (at 430.53 34.29 0)
+      (effects (font (size 1.27 1.27)) hide)
+    )
+    (pin "1")
+  )
   (symbol (lib_id "Connector_Generic:Conn_01x02") (at 315.595 177.8 0) (mirror y) (unit 1)
     (in_bom yes) (on_board yes) (fields_autoplaced)
@@
     (pin "1")
   )
+  (symbol (lib_id "power:+5V") (at 430.53 36.83 270) (mirror x) (unit 1)
+    (in_bom yes) (on_board yes)
+    (property "Reference" "#PWR?" (id 0) (at 426.72 36.83 0)
+      (effects (font (size 1.27 1.27)) hide)
+    )
+    (property "Value" "+5V" (id 1) (at 434.975 36.83 90))
+    (property "Footprint" "" (id 2) (at 430.53 36.83 0)
+      (effects (font (size 1.27 1.27)) hide)
+    )
+    (property "Datasheet" "" (id 3) (at 430.53 36.83 0)
+      (effects (font (size 1.27 1.27)) hide)
+    )
+    (pin "1")
+  )
   (symbol (lib_id "power:GND") (at 293.37 53.34 0) (mirror y) (unit 1)
     (in_bom yes) (on_board yes)
@@
       (reference "#PWR0136") (unit 1) (value "GND") (footprint "")
     )
+    (path "/15fcb7b1-ef4d-4c5b-847f-07ea1cbb9ecf"
+      (reference "#PWR?") (unit 1) (value "+3.3V") (footprint "")
+    )
+    (path "/96ea4fca-0370-42f9-8ba9-4f6e2f1c5a5b"
+      (reference "#PWR?") (unit 1) (value "+5V") (footprint "")
+    )
     (path "/820be99e-518a-4da7-b460-d2f0ce6373dc"

Commit message: #14 #15
Parts:
- added J19: 6437288-3, TE_6437288-3, symbol TE_6437288-3:6437288-3
- C10, C11, C12: footprint hellen-one-common:C0603 -> Capacitor_SMD:C_0603_1608Metric
Connections:
- net CAN_RX: now also J19.7 (7A)
- net CAN_TX: now also J19.6 (6A)
- net OUT0: now also J19.14 (14A)
- net OUT1: now also J19.15 (15A)
- net OUT2: now also J19.16 (16A)
- net OUT3: now also J19.17 (17A)
Other:
- moved on the sheet: C10, C11, C12, J18, U12

Commit message: #3
Parts:
- added F2: nSMD005, Fuse:Fuse_1206_3216Metric, symbol Device:Fuse
- added Q1: AO3400A, hellen-one-common:SOT-23, symbol hellen-one-common:MOSFET-N
- added R14: 4.7k, Resistor_SMD:R_0603_1608Metric, symbol Device:R
Connections:
- net GND: now also Q1.3 (S), R14.1
- net HALL0: now reaches U11.CN12_64 (PE0)
- net HALL0: now also Q1.1 (G), R14.2
- new net: F2.1, Q1.2 (D)
- new net OUT_HALL0: F2.2

Commit message: #3 #14 #16 #11 #17
Parts:
- removed J1, J2: Conn_01x16, TerminalBlock_Phoenix:TerminalBlock_Phoenix_MKDS-1,5-16-5.08_1x16_P5.08mm_Horizontal, symbol Connector_Generic:Conn_01x16
- removed J18: Conn_01x02, TerminalBlock_Phoenix:TerminalBlock_Phoenix_MKDS-1,5-2-5.08_1x02_P5.08mm_Horizontal, symbol Connector_Generic:Conn_01x02
- added F3, F4, F5, F6, F7, F8, F9: nSMD005, Fuse:Fuse_1206_3216Metric, symbol Device:Fuse
- added J1: 6437288-2, Connectors:6437288-2, symbol TE_6437288-2:6437288-2
- added Q2, Q3, Q4, Q5, Q6, Q7, Q8: AO3400A, hellen-one-common:SOT-23, symbol hellen-one-common:MOSFET-N
- added R15, R16, R17, R18, R19, R20, R21: 4.7k, Resistor_SMD:R_0603_1608Metric, symbol Device:R
- added R22: 1k, Resistor_SMD:R_0603_1608Metric, symbol Device:R
- added R23: 2k, Resistor_SMD:R_0603_1608Metric, symbol Device:R
- added R24, R28, R30, R38: 910, Resistor_SMD:R_0603_1608Metric, symbol Device:R
- added R25, R27, R29: 100, Resistor_SMD:R_0603_1608Metric, symbol Device:R
- added R26, R31, R32, R34, R35, R37, R39: 470, Resistor_SMD:R_0603_1608Metric, symbol Device:R
- added R33, R36: 330, Resistor_SMD:R_0603_1608Metric, symbol Device:R
- J19: footprint TE_6437288-3 -> kicad6-libraries:TE_6437288-3
- J3: value Conn_01x16 -> Conn_01x08; footprint TerminalBlock_Phoenix:TerminalBlock_Phoenix_MKDS-1,5-16-5.08_1x16_P5.08mm_Horizontal -> TerminalBlock_Phoenix:TerminalBlock_Phoenix_MKDS-1,5-8-5.08_1x08_P5.08mm_Horizontal; symbol Connector_Generic:Conn_01x16 -> Connector_Generic:Conn_01x08
Connections:
- net +12V: now also J19.37 (3B), J19.59 (25B)
- net CAN_H: now also J19.58 (24B)
- net CAN_L: now also J19.57 (23B)
- net CAN_RX: no longer J19.7 (7A)
- net CAN_TX: no longer J19.6 (6A)
- net GND: now also J19.60 (26B), Q2.3 (S), Q3.3 (S), Q4.3 (S), Q5.3 (S), Q6.3 (S), Q7.3 (S), Q8.3 (S), R15.1, R16.1, R17.1, R18.1, R19.1, R20.1, R21.1, R22.1, R23.1, R25.2, R27.2, R29.2, R31.2, R33.2, R35.2, R37.2, R38.2
- net OUT0: now also J19.49 (15B); no longer J19.14 (14A)
- net OUT1: now also J19.50 (16B); no longer J19.15 (15A)
- net OUT2: now also J19.51 (17B); no longer J19.16 (16A)
- net OUT3: now also J19.52 (18B); no longer J19.17 (17A)
- net TST1: now also J19.1 (1A)
- net TST10: now also J19.10 (10A)
- net TST11: now also J19.11 (11A)
- net TST12: now also J19.12 (12A)
- net TST13: now also J19.13 (13A)
- net TST14: now also J19.14 (14A)
- net TST15: now also J19.15 (15A)
- net TST16: now also J19.16 (16A)
- net TST17: now also J19.17 (17A)
- net TST18: now also J19.18 (18A)
- net TST19: now also J19.19 (19A)
- net TST2: now also J19.2 (2A)
- net TST20: now also J19.20 (20A)
- net TST21: now also J1.1 (1C)
- net TST22: now also J1.2 (2C)
- net TST23: now also J1.3 (3C)
- net TST24: now also J1.4 (4C)
- net TST25: now also J1.5 (5C)
- net TST26: now also J1.6 (6C)
- net TST27: now also J1.7 (7C)
- net TST28: now also J1.8 (8C)
- net TST29: now also J1.9 (9C)
- net TST3: now also J19.3 (3A)
- net TST30: now also J1.10 (10C)
- net TST31: now also J1.11 (11C)
- net TST32: now also J1.12 (12C)
- net TST33: now also J1.13 (13C); no longer J3.16 (Pin_16)
- net TST34: now also J1.14 (14C); no longer J3.15 (Pin_15)
- net TST35: now also J1.15 (15C); no longer J3.14 (Pin_14)
- net TST36: now also J1.16 (16C); no longer J3.13 (Pin_13)
- net TST37: now also J1.17 (17C); no longer J3.12 (Pin_12)
- net TST38: now also J1.18 (18C); no longer J3.11 (Pin_11)
- net TST39: now also J1.19 (19C); no longer J3.10 (Pin_10)
- net TST4: now also J19.4 (4A)
- net TST40: now also J1.20 (20C); no longer J3.9 (Pin_9)
- net TST5: now also J19.5 (5A)
- net TST6: now also J19.6 (6A)
- net TST7: now also J19.7 (7A)
- net TST8: now also J19.8 (8A)
- net TST9: now also J19.9 (9A)
- net 5V_1: now reaches J19.35 (1B)
- net 5V_1: now also R24.1, R26.1, R28.1, R30.1
- net 5V_2: now reaches J19.36 (2B)
- net 5V_2: now also R32.1, R34.1, R36.1, R39.1
- net at J19.39 (5B): now also R22.2
- net at J19.40 (6B): now also R23.2
- net REF1: now reaches J19.41 (7B)
- net REF1: now also R24.2, R25.1
- net REF2: now reaches J19.42 (8B)
- net REF2: now also R26.2, R27.1
- net REF3: now reaches J19.43 (9B)
- net REF3: now also R28.2, R29.1
- net REF4: now reaches J19.44 (10B)
- net REF4: now also R30.2, R31.1
- net REF5: now reaches J19.45 (11B)
- net REF5: now also R32.2, R33.1
- net REF6: now reaches J19.46 (12B)
- net REF6: now also R34.2, R35.1
- net REF7: now reaches J19.47 (13B)
- net REF7: now also R36.2, R37.1
- net REF8: now reaches J19.48 (14B)
- net REF8: now also R38.1, R39.2
- net OUT4: now reaches J19.53 (19B)
- net OUT5: now reaches J19.54 (20B)
- net OUT6: now reaches J19.55 (21B)
- net OUT7: now reaches J19.56 (22B)
- net HALL0_2: now reaches U11.CN12_40 (PE8)
- net HALL0_2: now also Q3.1 (G), R16.2
- net HALL0_1: now reaches U11.CN12_44 (PE7)
- net HALL0_1: now also Q2.1 (G), R15.2
- net HALL0_4: now reaches U11.CN12_47 (PE10)
- net HALL0_4: now also Q5.1 (G), R18.2
- net HALL0_6: now reaches U11.CN12_49 (PE12)
- net HALL0_6: now also Q7.1 (G), R20.2
- net HALL0_3: now reaches U11.CN12_52 (PE9)
- net HALL0_3: now also Q4.1 (G), R17.2
- net HALL0_7: now reaches U11.CN12_55 (PE13)
- net HALL0_7: now also Q8.1 (G), R21.2
- net HALL0_5: now reaches U11.CN12_56 (PE11)
- net HALL0_5: now also Q6.1 (G), R19.2
- net HALL0 renamed HALL0_0
- net OUT_HALL0 renamed OUT_HALL0_0
- new net: F5.1, Q4.2 (D)
- new net: F9.1, Q8.2 (D)
- new net: F8.1, Q7.2 (D)
- new net: F6.1, Q5.2 (D)
- new net: F7.1, Q6.2 (D)
- new net: F4.1, Q3.2 (D)
- new net: F3.1, Q2.2 (D)
- new net OUT_HALL0_1: F3.2
- new net OUT_HALL0_2: F4.2
- new net OUT_HALL0_3: F5.2
- new net OUT_HALL0_4: F6.2
- new net OUT_HALL0_5: F7.2
- new net OUT_HALL0_6: F8.2
- new net OUT_HALL0_7: F9.2
Other:
- note added: "0.5V"
- note added: "0.9V"
- note added: "1.3V"
- note added: "1.7V"
- note added: "2.1V"
- note added: "2.5V"
- note added: "2.9V"
- note added: "3.3V"
- title: (none) -> stim
- moved on the sheet: C10, C11, C12, F2, Q1, R14, U12

Commit message: #16 #17
Parts:
- added R40: 1k, Resistor_SMD:R_0603_1608Metric, symbol Device:R
- added R41: 2k, Resistor_SMD:R_0603_1608Metric, symbol Device:R
- added R42, R45, R58: 330, Resistor_SMD:R_0603_1608Metric, symbol Device:R
- added R43, R48: 910, Resistor_SMD:R_0603_1608Metric, symbol Device:R
- added R44, R46, R47, R59: 100, Resistor_SMD:R_0603_1608Metric, symbol Device:R
- added R49: 470, Resistor_SMD:R_0603_1608Metric, symbol Device:R
- R29: value 100 -> 330
Connections:
- net OUT4 is gone; now on net OUT_HALL0_4: J19.53 (19B)
- net OUT5 is gone; now on net OUT_HALL0_5: J19.54 (20B)
- net OUT6 is gone; now on net OUT_HALL0_6: J19.55 (21B)
- net OUT7 is gone; now on net OUT_HALL0_7: J19.56 (22B)
- net 5V_1: now also R39.1, R42.1, R44.1, R58.1; no longer R30.1
- net 5V_2: now also R30.1, R46.1, R47.1; no longer R36.1, R39.1
- net GND: now also R40.1, R41.1, R43.2, R45.2, R48.2, R49.2, R59.2
- net OUT0: no longer J19.49 (15B)
- net OUT1: no longer J19.50 (16B)
- net OUT2: no longer J19.51 (17B)
- net OUT3: no longer J19.52 (18B)
- net OUT_HALL0_0: now also J19.49 (15B)
- net OUT_HALL0_1: now also J19.50 (16B)
- net OUT_HALL0_2: now also J19.51 (17B)
- net OUT_HALL0_3: now also J19.52 (18B)
- net REF3: now also R58.2, R59.1; no longer R28.2, R29.1
- net REF4: now also R28.2, R29.1; no longer R30.2, R31.1
- net REF5: now also R30.2, R31.1; no longer R32.2, R33.1
- net REF6: now also R32.2, R33.1; no longer R34.2, R35.1
- net REF7: now also R34.2, R35.1; no longer R36.2, R37.1
- net REF8: now also R36.2, R37.1; no longer R38.1, R39.2
- net at J1.21 (21C): now also R40.2
- net at J1.22 (22C): now also R41.2
- net REF9: now reaches J1.23 (23C)
- net REF9: now also R38.1, R39.2
- net REF10: now reaches J1.24 (24C)
- net REF10: now also R42.2, R43.1
- net REF11: now reaches J1.25 (25C)
- net REF11: now also R44.2, R45.1
- net REF12: now reaches J1.26 (26C)
- net REF12: now also R46.2, R49.1
- net REF13: now reaches J1.27 (27C)
- net REF13: now also R47.2, R48.1
- net REF14: now reaches J1.28 (28C)
- net REF15: now reaches J1.29 (29C)
- net REF16: now reaches J1.30 (30C)
Other:
- note added: "1.2V"
- note added: "3.7V"
- note added: "3.8V"
- note added: "4.1V"
- note added: "4.5V"
- moved on the sheet: C10, C11, C12, J1, J19A, J19B, R22, R23, R24, R25, R26, R27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

Commit message: Трассированная плата + файл замены U11
Parts:
- added R50: 330, Resistor_SMD:R_0603_1608Metric, symbol Device:R
- added R51, R52, R53: 470, Resistor_SMD:R_0603_1608Metric, symbol Device:R
- added R54, R55: 910, Resistor_SMD:R_0603_1608Metric, symbol Device:R
- R34, R35: value 470 -> 100; LCSC C23179 -> C22775
- R37: value 470 -> 330; LCSC C23179 -> C23138
Connections:
- net 5V_1: now also R47.1, R50.1, R52.1, R54.1; no longer R39.1, R42.1, R44.1
- net 5V_2: now also R36.1, R39.1, R42.1, R44.1; no longer R47.1
- net GND: now also R51.2, R53.2, R55.2
- net REF10: now also R54.2, R55.1; no longer R42.2, R43.1
- net REF11: now also R50.2, R51.1; no longer R44.2, R45.1
- net REF12: now also R38.1, R39.2; no longer R46.2, R49.1
- net REF13: now also R42.2, R43.1; no longer R47.2, R48.1
- net REF14: now also R44.2, R45.1
- net REF15: now also R46.2, R49.1
- net REF16: now also R47.2, R48.1
- net REF9: now also R52.2, R53.1; no longer R38.1, R39.2
- no-connect marks 0 -> 19
Other:
- moved on the sheet: R38, R39, R42, R43, R44, R45, R46, R47, R48, R49
