File: digital_inputs/digital_inputs.kicad_sch (KiCad schematic)
At the start: 182 parts, among them J1 6437288-2, J10 Conn_01x01, J11 Conn_01x01, J12 Conn_01x01, J13 Conn_01x01, J14 Conn_01x01, J15 Conn_01x01, J16 Conn_01x01, J17 Conn_01x01, J18 Conn_02x05_Odd_Even, J19 6437288-3, J2 Conn_02x07_Odd_Even, J20 Conn_02x24_Odd_Even, J21 Conn_02x08_Odd_Even, J22 Conn_02x15_Odd_Even, J23 Conn_02x10_Odd_Even, J24 Conn_02x17_Odd_Even, J25 Conn_02x10_Odd_Even, J26 Conn_02x06_Odd_Even, J27 Conn_02x16_Odd_Even, J28 Conn_02x04_Odd_Even, J3 Conn_01x08, J4 Conn_01x01, J5 Conn_01x02, J6 Conn_01x04, J7 Conn_01x04, J8 Conn_01x04, J9 Conn_01x04, P1 Pad, P10 Pad, P11 Pad, P12 Pad, P13 Pad, P14 Pad, P15 Pad, P16 Pad, P17 Pad, P18 Pad, P19 Pad, P2 Pad, P3 Pad, P4 Pad, P5 Pad, P6 Pad, P7 Pad, P8 Pad, P9 Pad, Q1 AO3400A, Q2 AO3400A, Q3 AO3400A, Q4 AO3400A, Q5 AO3400A, Q6 AO3400A, Q7 AO3400A, Q8 AO3400A, Q9 PJM2319PSA, U1 OPA2192IDR, U10 ULN2003A, U11 OPA2192IDR, U12 TJA1051T-3, U13 TJA1051T-3, U2 CD4067BM96, U3 CD4067BM96, U4 CD4067BM96, U5 CD4067BM96, U6 CD4067BM96, U7 CD4067BM96, U8 TC4427, U9 TC4427

Commit message: Upd PCB
Parts:
- removed D5: BZV55C10, Diode_SMD:D_MiniMELF, symbol Diode:BZV55C10
- removed Q9: PJM2319PSA, Package_TO_SOT_SMD:SOT-23, symbol Transistor_FET:Si2319CDS
- removed R56, R62: DNP, Resistor_SMD:R_0402_1005Metric, symbol hellen1-wbo-rescue:R-Device
- removed R61: 13k, Resistor_SMD:R_0603_1608Metric, symbol Device:R
- added R56, R62: DNP, Resistor_SMD:R_0603_1608Metric, symbol Device:R
- CB1: footprint Button_Switch_SMD:SW_Push_SPST_NO_Alps_SKRK -> lib:RS601HL-1010011BB; LCSC C115357 -> C2885782
- J1: footprint Connectors:6437288-2 -> 6437288-2
Connections:
- net +12V: now also CB1.2
- net CAN2_H: now also R62.1
- net CAN2_L: now also R62.2
- net CAN_H: now also R56.1
- net CAN_L: now also R56.2
- net at F1.1: now also CB1.1; no longer CB1.2
Other:
- moved on the sheet: CB1

Commit message: Fix #41
Parts:
- J19: footprint kicad6-libraries:TE_6437288-3 -> TE_6437288-3; LCSC (none) -> C591769
Changed lines of the file:
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@@
       (effects (font (size 1.27 1.27)) (justify left bottom))
     )
-    (property "Footprint" "kicad6-libraries:TE_6437288-3" (at 229.87 308.61 0)
+    (property "Footprint" "TE_6437288-3" (at 229.87 308.61 0)
       (effects (font (size 1.27 1.27)) (justify left bottom) hide)
     )
@@
     (property "Comment" "6437288-3" (at 229.87 311.15 0)
       (effects (font (size 1.27 1.27)) (justify left bottom) hide)
+    )
+    (property "LCSC" "C591769" (at 236.22 314.96 0)
+      (effects (font (size 1.27 1.27)) hide)
     )
     (pin "1")
@@
       (effects (font (size 1.27 1.27)) (justify left bottom))
     )
-    (property "Footprint" "kicad6-libraries:TE_6437288-3" (at 229.87 209.55 0)
+    (property "Footprint" "TE_6437288-3" (at 229.87 209.55 0)
       (effects (font (size 1.27 1.27)) (justify left bottom) hide)
     )
@@
       (effects (font (size 1.27 1.27)) (justify left bottom) hide)
     )
-    (pin "1")
+    (property "LCSC" "C591769" (at 236.22 215.9 0)
+      (effects (font (size 1.27 1.27)) hide)
+    )
+    (pin "1")

Commit message: Rev D export
Parts:
- removed J18: Conn_02x05_Odd_Even, Connector_PinHeader_2.54mm:PinHeader_2x05_P2.54mm_Vertical, symbol Connector_Generic:Conn_02x05_Odd_Even
- removed J2: Conn_02x07_Odd_Even, Connector_PinHeader_2.54mm:PinHeader_2x07_P2.54mm_Vertical, symbol Connector_Generic:Conn_02x07_Odd_Even
- removed J20: Conn_02x24_Odd_Even, Connector_PinHeader_2.54mm:PinHeader_2x24_P2.54mm_Vertical, symbol Connector_Generic:Conn_02x24_Odd_Even
- added C17, C18: 10u, Capacitor_SMD:C_0805_2012Metric, symbol hellen-one-common:Cap
- added J20, J29: Conn_02x10_Odd_Even, Connector_PinHeader_2.54mm:PinHeader_2x10_P2.54mm_Vertical, symbol Connector_Generic:Conn_02x10_Odd_Even
- added J30: Conn_02x14_Odd_Even, Connector_PinHeader_2.54mm:PinHeader_2x16_P2.54mm_Vertical, symbol Connector_Generic:Conn_02x14_Odd_Even
- added U14: LM78M05_TO252, Package_TO_SOT_SMD:TO-252-2, symbol Regulator_Linear:LM78M05_TO252
Connections:
- net +12V: now also C17.2, J30.4 (VIN), U14.1 (VI)
- net +3.3V: now also J20.16 (+3V3)
- net +5V: now also J20.18 (+5V)
- net CAN_RX: now also J29.5 (PD0)
- net CAN_TX: now also J29.3 (PD1)
- net GND: now also C17.1, C18.1, J20.19 (GND), J20.20 (GND), J20.8 (GND), J29.19 (GND), J29.20 (GND), J29.8 (GND), J30.2 (GND), J30.29 (GND), U14.2 (GND)
- new net E5V: C18.2, J20.6 (E5V), U14.3 (VO)
- no-connect marks 199 -> 198
