File: digital_inputs.kicad_pcb (KiCad board)
At the start: 2 copper layers, 182.5 x 165 mm, 182 parts, among them J1 6437288-2, J10 Conn_01x01, J11 Conn_01x01, J12 Conn_01x01, J13 Conn_01x01, J14 Conn_01x01, J15 Conn_01x01, J16 Conn_01x01, J17 Conn_01x01, J19 6437288-3, J20 Conn_02x10_Odd_Even, J21 Conn_02x08_Odd_Even, J22 Conn_02x15_Odd_Even, J23 Conn_02x10_Odd_Even, J24 Conn_02x17_Odd_Even, J25 Conn_02x10_Odd_Even, J26 Conn_02x06_Odd_Even, J27 Conn_02x16_Odd_Even, J28 Conn_02x04_Odd_Even, J29 Conn_02x10_Odd_Even, J3 Conn_01x08, J30 Conn_02x14_Odd_Even, J4 Conn_01x01, J5 Conn_01x02, J6 Conn_01x04, J7 Conn_01x04, J8 Conn_01x04, J9 Conn_01x04, P1 Pad, P10 Pad, P11 Pad, P12 Pad, P13 Pad, P14 Pad, P15 Pad, P16 Pad, P17 Pad, P18 Pad, P19 Pad, P2 Pad, P3 Pad, P4 Pad, P5 Pad, P6 Pad, P7 Pad, P8 Pad, P9 Pad, Q1 AO3400A, Q2 AO3400A, Q3 AO3400A, Q4 AO3400A, Q5 AO3400A, Q6 AO3400A, Q7 AO3400A, Q8 AO3400A, U1 OPA2192IDR, U10 ULN2003A, U11 OPA2192IDR, U12 TJA1051T-3, U13 TJA1051T-3, U14 LM78M05_TO252, U2 CD4067BM96, U3 CD4067BM96, U4 CD4067BM96, U5 CD4067BM96, U6 CD4067BM96, U7 CD4067BM96, U8 TC4427, U9 TC4427

Commit message: #52
Parts:
- removed J5: Conn_01x02, TerminalBlock_Phoenix:TerminalBlock_Phoenix_MKDS-1,5-2-5.08_1x02_P5.08mm_Horizontal
- added J2: Barrel_Jack_Switch, Connector_BarrelJack:BarrelJack_GCT_DCJ200-10-A_Horizontal, F.Cu at (169.3, 196.7)
Routing:
- net Net-(F1-Pad2): track 4.43 -> 10.6 mm
Other:
- board text added: "Digital inputs rev E rusefi.com"
- board text removed: "Digital inputs rev D rusefi.com"
